File: hardware/av-board/av-board.kicad_sch (KiCad schematic)
At the start: 218 parts, among them J1 RCA Y, J10 2x20 socket, J2 RCA Pb, J3 RCA Pr, J4 RCA L, J5 RCA R, J6 HDMI-001, J9 2x20 socket, SW1 TS-1187A-B-A-B, SW2 TS-1187A-B-A-B, U1 ADV7842KBCZ-5, U10 TPD4E05U06DQAR, U2 ADV7511KSTZ, U3 PCM1808PWR, U4 TLV62569DBVR, U5 TPS7A7001DDAR, U6 TPS7A7001DDAR, U7 TPS7A7001DDAR, U8 TPD4E05U06DQAR, U9 TPD4E05U06DQAR, Y1 28.63636MHz 20pF

Commit message: Single pull-down resistors, SYNC_Y escape via, rail caps by their rail pad
From a round of free Freerouting trials (each variant routed on fpga, DRC'd, failures counted
over several runs):

- The unused SDRAM port's 18 pull-downs are single 0402s by the ADV7842's right side. With
  4-resistor arrays two to five of them failed in every run on both routers (four lines meeting a
  0.5 mm-pitch array in order, in the board's tightest corner); with singles, rarely one.
- SYNC_Y (J15) takes an escape via like the pull-down balls: it failed in nearly every run on
  F.Cu under the analog inputs' terminations, and not once with the via.
- A rail cap is placed where its rail pad (0.3 mm in) is over its plane, not its whole footprint:
  all 69 now sit on their planes (three were off). The plane fanout puts a rail pad's via only
  where the via itself lands on the plane (one off it connected nothing), tries 16 directions up
  to 2.5 mm, and names the pads left without one (their caps are joined by a routed track).
- CVDD's filter FL3 sits beside FL6, a short branch off FL4's 1V8A.

Tried and dropped: a wider free ring above the analog edge, more room round each rail cap,
reserved via spots, pull-down arrays on B.Cu or further out, vias for REFP/REFN, turning U5/U7.

Freerouting on this board leaves 2-7 short connections depending on the run. ERC clean,
schematic = board.py, DRC: only the unrouted connections.

Co-Authored-By: Claude Opus 5.5 <noreply@anthropic.com>
Parts:
- removed RN6, RN7, RN8, RN9: 4.7k, lcsc:RES-ARRAY-SMD_0402-8P-L2.0-W1.0-BL, symbol lcsc:4D02WGJ0472TCE
- added R52, R53, R54, R55, R67: 10k, Resistor_SMD:R_0402_1005Metric, symbol Device:R
- added R56, R57, R58, R59: 51, Resistor_SMD:R_0402_1005Metric, symbol Device:R
- added R60: 887, Resistor_SMD:R_0402_1005Metric, symbol Device:R
- added R61, R62, R63, R64, R65, R66: 2k, Resistor_SMD:R_0402_1005Metric, symbol Device:R
- R33, R34, R35, R36, R37, R38, R39: value 10k -> 4.7k; LCSC C25744 -> C25900
- R40, R41, R42, R43: value 51 -> 4.7k; LCSC C25125 -> C25900
- R44: value 887 -> 4.7k; LCSC C55968414 -> C25900
- R45, R46, R47, R48: value 2k -> 4.7k; LCSC C4109 -> C25900
- R49, R50: value 2k -> 10k; LCSC C4109 -> C25744
- R51: Note 0 V on HPD with no sink [HWG 6.1.4: 10 k +-10 %] -> (none)
Connections:
- net 3V3: now also R61.1, R62.1, R63.1; no longer R45.1, R46.1, R47.1
- net AUD_DIV_L: now also R52.2, R53.1; no longer R36.2, R37.1
- net AUD_DIV_R: now also R54.2, R55.1; no longer R38.2, R39.1
- net FMT: now also R51.1; no longer R35.1
- net GND: now also R36.2, R38.2, R40.2, R41.2, R42.2, R43.2, R45.2, R46.2, R47.2, R49.2, R50.2, R53.2, R55.2, R60.2, R64.2, R67.2
- net HDMI_5V: now also R65.1, R66.1; no longer R49.1, R50.1
- net HDMI_HPD: now also R67.1; no longer R51.1
- net HDMI_SCL: now also R65.2; no longer R49.2
- net HDMI_SDA: now also R66.2; no longer R50.2
- net MD0: now also R49.1; no longer R33.1
- net MD1: now also R50.1; no longer R34.1
- net OUT_I2S0: now also R59.1; no longer R43.1
- net OUT_INT: now also R63.2; no longer R47.2
- net OUT_LRCLK: now also R58.1; no longer R42.1
- net OUT_MCLK: now also R56.1; no longer R40.1
- net OUT_PD: now also R64.1; no longer R48.1
- net OUT_SCL: now also R61.2; no longer R45.2
- net OUT_SCLK: now also R57.1; no longer R41.1
- net OUT_SDA: now also R62.2; no longer R46.2
- net PD_SDRAM_DQ0: now also R31.1
- net PD_SDRAM_DQ1: now also R32.1
- net PD_SDRAM_DQ10: now also R41.1
- net PD_SDRAM_DQ11: now also R42.1
- net PD_SDRAM_DQ12: now also R43.1
- net PD_SDRAM_DQ13: now also R44.1
- net PD_SDRAM_DQ14: now also R45.1
- net PD_SDRAM_DQ15: now also R46.1
- net PD_SDRAM_DQ2: now also R33.1
- net PD_SDRAM_DQ3: now also R34.1
- net PD_SDRAM_DQ4: now also R35.1
- net PD_SDRAM_DQ5: now also R36.1
- net PD_SDRAM_DQ6: now also R37.1
- net PD_SDRAM_DQ7: now also R38.1
- net PD_SDRAM_DQ8: now also R39.1; no longer R32.1
- net PD_SDRAM_DQ9: now also R40.1
- net PD_SDRAM_LDQS: now also R47.1; no longer R31.1
- net PD_SDRAM_UDQS: now also R48.1
- net RCA_L: now also R52.1; no longer R36.1
- net RCA_R: now also R54.1; no longer R38.1
- net R_EXT: now also R60.1; no longer R44.1
- net TX_I2S0: now also R59.2; no longer R43.2
- net TX_LRCLK: now also R58.2; no longer R42.2
- net TX_MCLK: now also R56.2; no longer R40.2
- net TX_SCLK: now also R57.2; no longer R41.2
Other:
- moved on the sheet: C100, C101, C102, C103, C41, C42, C43, C44, C45, C46, C47, C48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
