File: hardware/av-board/rev-a/av-board-a.kicad_sch (KiCad schematic)
At the start: 230 parts, among them J1 RCA Y, J10 2x20 socket, J2 RCA Pb, J3 RCA Pr, J4 RCA L, J5 RCA R, J6 HDMI-001, J9 2x20 socket, SW1 TS-1187A-B-A-B, SW2 TS-1187A-B-A-B, U1 ADV7842KBCZ-5, U10 TPD4E05U06DQAR, U2 ADV7511KSTZ, U3 PCM1808PWR, U4 TLV62569DBVR, U5 TPS7A7001DDAR, U6 TPS7A7001DDAR, U7 TPS7A7001DDAR, U8 TPD4E05U06DQAR, U9 TPD4E05U06DQAR, Y1 28.63636MHz 20pF

Commit message: AV board: revisions in rev-a/, shared generators in kit/
The board moves to hardware/av-board/rev-a/ (av-board-a.*): its board.py and gen_pcb.py keep
only what is rev A's own. What a next revision reuses goes to kit/: parts.py (the part
record, two-pin parts and LCSC numbers, the Console headers), pcbkit.py (the placer, fanout,
rules, planes, routing passes and silkscreen, as a Layout class a revision subclasses with
hooks for its chips), and the tools, which now take the revision (kit/gen_sch.py rev-a).

Rev A regenerates exactly as before: the same parts and nets, placement, fanout copper,
zones and silkscreen, and the same Gerbers, drills, BOM and CPL (only the file names carry
the revision).

Co-Authored-By: Claude Opus 5.5 <noreply@anthropic.com>
Other:
- title: Tang Console AV board -> Tang Console AV board rev A
