File: hardware/av-board/rev-a/av-board-a.kicad_pcb (KiCad board)
At the start: 6 copper layers, 94.6 x 69.4 mm, 234 parts, among them J1 RCA Y, J10 2x20 socket, J2 RCA Pb, J3 RCA Pr, J4 RCA L, J5 RCA R, J6 HDMI-001, J9 2x20 socket, SW1 TS-1187A-B-A-B, SW2 TS-1187A-B-A-B, U1 ADV7842KBCZ-5, U10 TPD4E05U06DQAR, U2 ADV7511KSTZ, U3 PCM1808PWR, U4 TLV62569DBVR, U5 TPS7A7001DDAR, U6 TPS7A7001DDAR, U7 TPS7A7001DDAR, U8 TPD4E05U06DQAR, U9 TPD4E05U06DQAR, Y1 28.63636MHz 20pF

Commit message: AV boards: the last complete, valid design of each revision; decoupling at the pins
Each revision's board, schematic, fab files and renders are its last complete
route: DRC clean, no unconnected items, ERC clean, the board equal to its
schematic part for part (pads, values, footprints; only the mounting holes
H1-H4 have no symbol).

- Rev A: the silkscreen pass (labels clear of pads, texts and part bodies);
  copper unchanged.
- Rev B: the previous route with the silkscreen pass. Its schematic stays the
  one it was routed from: board.py now numbers eight capacitors the other way
  round, and its placement fixes (below) are not routed yet, the routes on the
  new placement having left 1 and 3 connections (review.md, Status).
- C-A: routed again on the fixed placement (try-ca-p1), the copper the router
  laid twice over taken up (218 segments).
- C-B: S/PDIF on rev B's 5-pin header instead of the coax jack, the HDMI
  receptacle next to the RCAs, the board 100 x 100 mm; routed again on the
  fixed placement (try-cb-p3). 5.4 mm of copper laid side by side in five
  nets is left (rev-c/review.md).

The review found decoupling not at the pins on every board (ADV7511 9-25 mm,
DP159 6-13 mm, the bucks' input capacitor by EN, the LDOs' capacitors, the
clock LDOs 73-80 mm from their chip) and C's VBUS_IN 0.25 mm wide for 2 A:
- parts.py: Part.at = "REF.PAD", the one pad a capacitor or filter serves;
  circuits, carrier.py and board.py name it for every regulator and supply pin
- pcbkit.py placer: ESD parts first, then small chips, then the at= capacitors
  and bias parts in board.py order; mean pin-to-capacitor distance on the
  placements: rev B 8.1 -> 3.6 mm, C-A 6.3 -> 3.3, C-B 5.5 -> 3.4
- rev C: VBUS_IN 0.7/1.2 mm into the TVS and fuse; rev B and C: the coax
  slicer placed first (SPDIF_AC a bias net); rev B: the buck U4 turned over

Kit: the silkscreen pass (labels clear of pads, texts, parts and the SOM,
reserved in the placer); prune takes up copper lying on another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
Changed lines of the file:
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@@
 		(at 164 76)
 		(property "Reference" "SW1"
-			(at 0 -3.375 0)
+			(at 0 3.375 0)
 			(layer "F.SilkS")
 			(effects
@@
 		(layer "Edge.Cuts")
 	)
-	(gr_text "tang-av-scaler AV board rev A"
-		(at 116.5 88.4 0)
+	(gr_text "R"
+		(at 90.05 39.099999 0)
 		(layer "F.SilkS")
 		(effects
 			(font
-				(size 1.2 1.2)
-				(thickness 0.18)
+				(size 1 1)
+				(thickness 0.15)
 			)
+			(justify left)
 		)
 	)
-	(gr_text "HDMI"
-		(at 162.42 71.8 0)
+	(gr_text "tang-av-scaler AV board rev A"
+		(at 116.5 88.4 0)
 		(layer "F.SilkS")
 		(effects
@@
 		)
 	)
-	(gr_text "L"
-		(at 75.8 29.3 90)
+	(gr_text "HDMI"
+		(at 162.42 71.8 0)
 		(layer "F.SilkS")
 		(effects
 			(font
-				(size 1.4 1.4)
+				(size 1.2 1.2)
 				(thickness 0.18)
 			)
 		)
 	)
-	(gr_text "R"
-		(at 75.8 42.3 90)
+	(gr_text "L"
+		(at 89.55 29.3 0)
 		(layer "F.SilkS")
 		(effects
@@
 				(thickness 0.18)
 			)
+			(justify left)
 		)
 	)
 	(gr_text "Y"
-		(at 75.8 55.3 90)
+		(at 90.05 55.3 0)
 		(layer "F.SilkS")
 		(effects
@@
 				(thickness 0.18)
 			)
+			(justify left)
 		)
 	)
 	(gr_text "Pb"
-		(at 75.8 68.3 90)
+		(at 90.05 68.3 0)
 		(layer "F.SilkS")
 		(effects
@@
 				(thickness 0.18)
 			)
+			(justify left)
 		)
 	)
 	(gr_text "Pr"
-		(at 75.8 81.3 90)
+		(at 90.05 81.3 0)
 		(layer "F.SilkS")
 		(effects
@@
 				(thickness 0.18)
 			)
+			(justify left)
 		)
 	)
