File: hardware/av-board/rev-b/av-board-b.kicad_sch (KiCad schematic)
At the start: 172 parts, among them J1 RCA Y, J10 2x20 socket, J2 RCA Pb, J3 RCA Pr, J4 RCA L, J5 RCA R, J6 HDMI-001, J9 2x20 socket, SW1 TS-1187A-B-A-B, SW2 TS-1187A-B-A-B, U1 ADV7181DBCPZ-RL, U10 TPD4E05U06DQAR, U2 ADV7511KSTZ, U3 PCM1808PWR, U4 TLV62569DBVR, U5 TPS7A7001DDAR, U6 TPS7A7001DDAR, U7 TPS7A7001DDAR, U8 TPD4E05U06DQAR, U9 TPD4E05U06DQAR, Y1 28.63636MHz 20pF

Commit message: Rev B routed: DRC clean, fab files
Freerouting connected every net on four layers over the locked fanout; the TMDS pairs were
then laid again pair-wise on the outer layers with mazeroute.py (Freerouting had taken two
through In2, which has no close ground on this stack), skew 1.2-5.1 mm. DRC: no errors, no
unconnected items. fab/: Gerbers, BOM (46 lines), CPL (172 parts, 14 on the bottom). ERC
clean, schematic = board.py.

Co-Authored-By: Claude Opus 5.5 <noreply@anthropic.com>
Parts:
- C28, C29: value 30p -> 33p; LCSC C1570 -> C1562
- J1, J2, J4: symbol lcsc:RCJ-011 -> lcsc:RCJ-014; LCSC C4992678 -> C4991844; Note black RCJ-01x -> yellow RCJ-01x
- R53, R54, R55, R56: value 51 -> 49.9; LCSC C25125 -> C25120
Changed lines of the file:
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@@
 )
   (symbol
-    (lib_id "lcsc:RCJ-011")
+    (lib_id "lcsc:RCJ-014")
     (at 749.3 36.83 0)
     (unit 1)
@@
         (font (size 1.27 1.27))
         (hide yes)))
-    (property "LCSC" "C4992678"
+    (property "LCSC" "C4991844"
       (at 749.3 36.83 0)
       (effects
         (font (size 1.27 1.27))
         (hide yes)))
-    (property "Note" "black RCJ-01x"
+    (property "Note" "yellow RCJ-01x"
       (at 749.3 36.83 0)
       (effects
@@
 )
   (symbol
-    (lib_id "lcsc:RCJ-011")
+    (lib_id "lcsc:RCJ-014")
     (at 821.69 36.83 0)
     (unit 1)
@@
         (font (size 1.27 1.27))
         (hide yes)))
-    (property "LCSC" "C4992678"
+    (property "LCSC" "C4991844"
       (at 821.69 36.83 0)
       (effects
         (font (size 1.27 1.27))
         (hide yes)))
-    (property "Note" "black RCJ-01x"
+    (property "Note" "yellow RCJ-01x"
       (at 821.69 36.83 0)
       (effects
@@
       (effects
         (font (size 1.27 1.27))))
-    (property "Value" "30p"
+    (property "Value" "33p"
       (at 821.69 138.43 0)
       (effects
@@
         (font (size 1.27 1.27))
         (hide yes)))
-    (property "LCSC" "C1570"
+    (property "LCSC" "C1562"
       (at 821.69 130.81 0)
       (effects
@@
       (effects
         (font (size 1.27 1.27))))
-    (property "Value" "30p"
+    (property "Value" "33p"
       (at 843.28 138.43 0)
       (effects
@@
         (font (size 1.27 1.27))
         (hide yes)))
-    (property "LCSC" "C1570"
+    (property "LCSC" "C1562"
       (at 843.28 130.81 0)
       (effects
@@
 )
   (symbol
-    (lib_id "lcsc:RCJ-011")
+    (lib_id "lcsc:RCJ-014")
     (at 1009.65 71.12 0)
     (unit 1)
@@
         (font (size 1.27 1.27))
         (hide yes)))
-    (property "LCSC" "C4992678"
+    (property "LCSC" "C4991844"
       (at 1009.65 71.12 0)
       (effects
         (font (size 1.27 1.27))
         (hide yes)))
-    (property "Note" "black RCJ-01x"
+    (property "Note" "yellow RCJ-01x"
       (at 1009.65 71.12 0)
       (effects
@@
       (effects
         (font (size 1.27 1.27))))
-    (property "Value" "51"
+    (property "Value" "49.9"
       (at 1155.7 189.23 0)
       (effects
@@
         (font (size 1.27 1.27))
         (hide yes)))
-    (property "LCSC" "C25125"
+    (property "LCSC" "C25120"
       (at 1155.7 181.61 0)
       (effects
@@
       (effects
         (font (size 1.27 1.27))))
-    (property "Value" "51"
+    (property "Value" "49.9"
       (at 1186.18 189.23 0)
       (effects
@@
         (font (size 1.27 1.27))
         (hide yes)))
-    (property "LCSC" "C25125"
+    (property "LCSC" "C25120"
       (at 1186.18 181.61 0)
       (effects
@@
       (effects
         (font (size 1.27 1.27))))
-    (property "Value" "51"
+    (property "Value" "49.9"
       (at 1219.2 189.23 0)
       (effects
@@
         (font (size 1.27 1.27))
         (hide yes)))
-    (property "LCSC" "C25125"
+    (property "LCSC" "C25120"
       (at 1219.2 181.61 0)
       (effects
@@
       (effects
         (font (size 1.27 1.27))))
-    (property "Value" "51"
+    (property "Value" "49.9"
       (at 1250.95 189.23 0)
       (effects
@@
         (font (size 1.27 1.27))
         (hide yes)))
-    (property "LCSC" "C25125"
+    (property "LCSC" "C25120"
       (at 1250.95 181.61 0)
       (effects

Commit message: Rev B: SMT on the top only, resistor arrays, a BOM without the RCA jacks
Every SMT part is now on the top (only the through-hole J9/J10 sockets sit underneath), so
JLCPCB assembles one side. To make room for the ADV7181D decoupling on the top, the three
runs of four pixel pins get 4 x 0402 33 R arrays at the pins own 0.5 mm pitch, in line with
them (163 parts, from 172); the band between the chip and its resistors is kept for the lines
and each supply pin 100 nF is placed first (2.7-4.3 mm from its pin).

gen_fab.py writes a BOM + CPL per assembly variant (VARIANTS in board.py); rev B hand-jacks
leaves J1-J5 for soldering by hand. Same Gerbers.

The routing flow does the hand steps now: a post_route hook (rev B: the TMDS pairs ripped up
and laid pair-wise on the outer layers), then finish_unconnected (DRC unconnected list ->
copper islands -> nearest pad pair -> mazeroute.py). mazeroute keeps 10 um of slack over the
clearance and its new vias clear of its own nets drills. snap.py frames on the outline.

DRC: no errors, no unconnected items. ERC clean, schematic = board.py.

Co-Authored-By: Claude Opus 5.5 <noreply@anthropic.com>
Parts:
- removed R53, R54, R55, R56: 49.9, Resistor_SMD:R_0402_1005Metric, symbol Device:R
- removed R57: 887, Resistor_SMD:R_0402_1005Metric, symbol Device:R
- removed R58, R59, R60, R61, R62, R63: 2k, Resistor_SMD:R_0402_1005Metric, symbol Device:R
- removed R64: 10k, Resistor_SMD:R_0402_1005Metric, symbol Device:R
- added RN1, RN2, RN3: 33, lcsc:RES-ARRAY-SMD_0402-8P-L2.0-W1.0-BL, symbol lcsc:4D02WGJ0750TCE
- R25, R26, R28, R29, R30: value 33 -> 4.7k; LCSC C25105 -> C25900
- R27: value 33 -> 4.7k; LCSC C25105 -> C25900; Note (none) -> held in reset until the FPGA drives it (5 ms low minimum [D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
- R31, R32, R33, R34, R35, R36: value 33 -> 10k; LCSC C25105 -> C25744
- R37, R38, R40: value 4.7k -> 10k; LCSC C25900 -> C25744
- R39: value 4.7k -> 10k; LCSC C25900 -> C25744; Note held in reset until the FPGA drives it (5 ms low minimum [D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 -> (none)
- R41, R42: value 4.7k -> 49.9; LCSC C25900 -> C25120
- R43, R44: value 10k -> 49.9; LCSC C25744 -> C25120
- R45: value 10k -> 887; LCSC C25744 -> C55968414
- R46, R47, R48, R49, R50, R51: value 10k -> 2k; LCSC C25744 -> C4109
- R52: Note (none) -> 0 V on HPD with no sink [HWG 6.1.4: 10 k +-10 %]
Connections:
- net 3V3: now also R25.1, R26.1, R46.1, R47.1, R48.1; no longer R37.1, R38.1
- net ALSB: now also R29.2; no longer R41.2
- net AUD_DIV_L: now also R37.2, R38.1; no longer R49.2, R50.1
- net AUD_DIV_R: now also R39.2, R40.1; no longer R51.2, R52.1
- net AV_C0: now also R21.1; no longer R32.1
- net AV_C1: now also R20.1; no longer R31.1
- net AV_C2: now also RN3.3; no longer R30.1
- net AV_C3: now also RN3.2; no longer R29.1
- net AV_C4: now also RN3.1; no longer R28.1
- net AV_C5: now also R19.1; no longer R27.1
- net AV_C6: now also R18.1; no longer R26.1
- net AV_C7: now also R17.1; no longer R25.1
- net AV_DE: now also R24.1; no longer R36.1
- net AV_DVDDIO: now also R28.1, R29.1, R30.1; no longer R40.1, R41.1, R42.1
- net AV_HS: now also R22.1; no longer R34.1
- net AV_LLC: now also RN3.4; no longer R33.1
- net AV_VS: now also R23.1; no longer R35.1
- net AV_Y0: now also RN2.4; no longer R24.1
- net AV_Y1: now also RN2.3; no longer R23.1
- net AV_Y2: now also RN2.2; no longer R22.1
- net AV_Y3: now also RN2.1; no longer R21.1
- net AV_Y4: now also RN1.4; no longer R20.1
- net AV_Y5: now also RN1.3; no longer R19.1
- net AV_Y6: now also RN1.2; no longer R18.1
- net AV_Y7: now also RN1.1; no longer R17.1
- net FMT: now also R36.1; no longer R48.1
- net GND: now also R27.2, R31.2, R32.2, R33.2, R34.2, R35.2, R36.2, R38.2, R40.2, R49.2; no longer R39.2, R43.2, R44.2, R46.2, R47.2, R48.2, R50.2
- net HDMI_5V: now also R50.1, R51.1
- net HDMI_HPD: now also R52.1
- net HDMI_SCL: now also R50.2
- net HDMI_SDA: now also R51.2
- net IN_C0: now also R21.2; no longer R32.2
- net IN_C1: now also R20.2; no longer R31.2
- net IN_C2: now also RN3.6; no longer R30.2
- net IN_C3: now also RN3.7; no longer R29.2
- net IN_C4: now also RN3.8; no longer R28.2
- net IN_C5: now also R19.2; no longer R27.2
- net IN_C6: now also R18.2; no longer R26.2
- net IN_C7: now also R17.2; no longer R25.2
- net IN_DE: now also R24.2; no longer R36.2
- net IN_HS: now also R22.2; no longer R34.2
- net IN_INT: now also R28.2; no longer R40.2
- net IN_LLC: now also RN3.5; no longer R33.2
- net IN_RESET_N: now also R27.1; no longer R39.1
- net IN_SCL: now also R25.2; no longer R37.2
- net IN_SDA: now also R26.2; no longer R38.2
- net IN_VS: now also R23.2; no longer R35.2
- net IN_Y0: now also RN2.5; no longer R24.2
- net IN_Y1: now also RN2.6; no longer R23.2
- net IN_Y2: now also RN2.7; no longer R22.2
- net IN_Y3: now also RN2.8; no longer R21.2
- net IN_Y4: now also RN1.5; no longer R20.2
- net IN_Y5: now also RN1.6; no longer R19.2
- net IN_Y6: now also RN1.7; no longer R18.2
- net IN_Y7: now also RN1.8; no longer R17.2
- net MD0: now also R34.1; no longer R46.1
- net MD1: now also R35.1; no longer R47.1
- net OUT_I2S0: now also R44.1
- net OUT_INT: now also R48.2
- net OUT_LRCLK: now also R43.1
- net OUT_MCLK: now also R41.1
- net OUT_PD: now also R49.1
- net OUT_SCL: now also R46.2
- net OUT_SCLK: now also R42.1
- net OUT_SDA: now also R47.2
- net PD_FB: now also R31.1; no longer R43.1
- net PD_HS_IN_CS_IN: now also R32.1; no longer R44.1
- net PD_VS_IN: now also R33.1; no longer R45.1
- net PWRDWN: now also R30.2; no longer R42.2
- net RCA_L: now also R37.1; no longer R49.1
- net RCA_R: now also R39.1; no longer R51.1
- net R_EXT: now also R45.1
- net TX_I2S0: now also R44.2
- net TX_LRCLK: now also R43.2
- net TX_MCLK: now also R41.2
- net TX_SCLK: now also R42.2
Other:
- moved on the sheet: C44, C45, C46, C47, C48, C49, C50, C51, C52, C53, C54, C55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

Commit message: Rev B reviewed against every data sheet; supplies, stack-up and TMDS fixed
review.md: each part against its document, for margin, not just limits. Fixed:
- Supply sequencing: the ADV7181D allows 3.3 V at most 2 V above and 0.3 V below the 1.8 V
  rails [DS Table 5]; rev A RC enable put 3V3 30 ms ahead. Now buck -> 3V6 -> 3V3 LDO ->
  1.8 V LDOs fed and enabled by 3V3, plus a B5819W clamp 1V8A -> 3V3 for power-down. The 3V3
  LDO runs from 3.6 V (0.17 W, was 0.94 W).
- Ferrites: the 0.2 A / 0.45 R beads dropped AVDD under 3.15 V at the LDO low limit;
  BLM18PG121SN1D (2 A, 50 mR), a basic part.
- Crystal: YXC X50322863636MSB2GI (476 in stock, +-10 ppm) for the 68-in-stock TXM.
- Stack-up: In2 a second ground plane, signals on F/B only, each over its own plane (B.Cu had
  no plane closer than 1.3 mm) [HWG 7.2].
- TMDS: the pairs are laid by the generator on F.Cu, 0.25/0.25 mm at the pins 0.5 mm pitch
  (103 R), coupled pin to connector, no vias, 0.83 mm intra-pair skew; a corridor kept free;
  the pins between the pairs escape inwards under the package.
- R_EXT 2.2 mm from its pin; video inputs get a TPD4E05U06.

pcbkit: INNER_GND, ROUTE_LAYERS, MIN_VIA, TMDS geometry per revision, via sizes, pad-level
fanout skips; session() restores locked vias sizes (KiCad import resets them).

DRC: no errors, no unconnected items. ERC clean, schematic = board.py. Rev A unchanged.

Co-Authored-By: Claude Opus 5.5 <noreply@anthropic.com>
Parts:
- removed C77: 100n, Capacitor_SMD:C_0402_1005Metric, symbol Device:C
- removed R52: 10k, Resistor_SMD:R_0402_1005Metric, symbol Device:R
- added D1: B5819W, Diode_SMD:D_SOD-123, symbol Device:D_Schottky
- added U11: TPD4E05U06DQAR, lcsc:USON-10_L2.5-W1.0-P0.50-BL, symbol lcsc:TPD4E05U06DQAR_C138714
- C10: value 470n -> 10u; footprint Capacitor_SMD:C_0603_1608Metric -> Capacitor_SMD:C_0805_2012Metric; LCSC C1623 -> C15850
- C12, C15: value 10u -> 220p; footprint Capacitor_SMD:C_0805_2012Metric -> Capacitor_SMD:C_0402_1005Metric; LCSC C15850 -> C1530
- C13: value 220p -> 10u; footprint Capacitor_SMD:C_0402_1005Metric -> Capacitor_SMD:C_0805_2012Metric; LCSC C1530 -> C15850
- C16: value 220p -> 10u; footprint Capacitor_SMD:C_0402_1005Metric -> Capacitor_SMD:C_0603_1608Metric; LCSC C1530 -> C19702
- C23, C32, C35, C38, C40, C57, C59: value 10u -> 100n; footprint Capacitor_SMD:C_0603_1608Metric -> Capacitor_SMD:C_0402_1005Metric; LCSC C19702 -> C1525
- C26: value 100n -> 1n; LCSC C1525 -> C1523
- C27: value 1n -> 33p; LCSC C1523 -> C1562
- C29: value 33p -> 100n; LCSC C1562 -> C1525
- C31, C39, C56, C58, C60: value 100n -> 10u; footprint Capacitor_SMD:C_0402_1005Metric -> Capacitor_SMD:C_0603_1608Metric; LCSC C1525 -> C19702
- C33, C36, C44, C46, C48, C50, C52, C54: value 100n -> 10n; LCSC C1525 -> C15195
- C34, C37: value 10n -> 10u; footprint Capacitor_SMD:C_0402_1005Metric -> Capacitor_SMD:C_0603_1608Metric; LCSC C15195 -> C19702
- C41: value 100n -> 82n; LCSC C1525 -> C277511
- C42: value 82n -> 10n; LCSC C277511 -> C15195
- C43, C45, C47, C49, C51, C53, C55: value 10n -> 100n; LCSC C15195 -> C1525
- C6: value 220p -> 6.8p; LCSC C1530 -> C1576
- C61: value 10u -> 220p; footprint Capacitor_SMD:C_0603_1608Metric -> Capacitor_SMD:C_0402_1005Metric; LCSC C19702 -> C1530
- C62, C64: value 220p -> 1u; footprint Capacitor_SMD:C_0402_1005Metric -> Capacitor_SMD:C_0603_1608Metric; LCSC C1530 -> C15849
- C63: value 1u -> 220p; footprint Capacitor_SMD:C_0603_1608Metric -> Capacitor_SMD:C_0402_1005Metric; LCSC C15849 -> C1530
- C65: value 1u -> 100n; footprint Capacitor_SMD:C_0603_1608Metric -> Capacitor_SMD:C_0402_1005Metric; LCSC C15849 -> C1525
- C7: value 4.7u -> 10u; LCSC C1779 -> C15850
- C9: value 6.8p -> 220p; LCSC C1576 -> C1530
- FB1, FB2, FB3, FB4, FB5: value 600R -> 120R; LCSC C1002 -> C14709
- R10, R8: value 78.7k -> 30.1k; LCSC C67239 -> C29402
- R11: value 30.1k -> 75; footprint Resistor_SMD:R_0402_1005Metric -> Resistor_SMD:R_0603_1608Metric; LCSC C29402 -> C4275
- R14: value 75 -> 1M; footprint Resistor_SMD:R_0603_1608Metric -> Resistor_SMD:R_0402_1005Metric; LCSC C4275 -> C26083
- R15: value 1M -> 1.69k; LCSC C26083 -> C25870
- R16: value 1.69k -> 33; LCSC C25870 -> C25105
- R24: value 33 -> 4.7k; LCSC C25105 -> C25900
- R26: Note (none) -> held in reset until the FPGA drives it (5 ms low minimum [D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
- R27: Note held in reset until the FPGA drives it (5 ms low minimum [D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 -> (none)
- R3: value 169k -> 499k; LCSC C25758 -> C25793
- R30: value 4.7k -> 10k; LCSC C25900 -> C25744
- R4: value 30.1k -> 100k; LCSC C29402 -> C25741
- R40: value 10k -> 49.9; LCSC C25744 -> C25120
- R44: value 49.9 -> 887; LCSC C25120 -> C55968414
- R45: value 887 -> 2k; LCSC C55968414 -> C4109
- R5: value 316k -> 169k; LCSC C25777 -> C25758
- R51: value 2k -> 10k; LCSC C4109 -> C25744; Note (none) -> 0 V on HPD with no sink [HWG 6.1.4: 10 k +-10 %]
- R6: value 100k -> 30.1k; LCSC C25741 -> C29402
- R7: value 100k -> 78.7k; LCSC C25741 -> C67239
- R9: value 30.1k -> 78.7k; LCSC C29402 -> C67239
- Y1: LCSC C362486 -> C112564
Connections:
- net +5V: no longer C7.1, U5.2 (EN), U5.3 (IN)
- net 1V8A: now also C11.1, R7.1, D1.2 (A); no longer C13.1, R8.1
- net 1V8B: now also C14.1, R9.1; no longer C16.1, R10.1
- net 3V3: now also C10.1, C13.1, C59.1, C75.1, C8.1, C9.1, R24.1, R45.1, R5.1, U6.2 (EN), U6.3 (IN), U7.2 (EN), U7.3 (IN), D1.1 (K); no longer C5.1, C6.1, C61.1, C76.1, R26.1, R3.1, R48.1
- net 5VA: now also C57.1; no longer C59.1
- net AIN_PB: now also C24.2; no longer C25.2
- net AIN_PR: now also C25.2; no longer C26.2
- net AIN_Y: now also C23.2; no longer C24.2
- net ALSB: now also R28.2; no longer R29.2
- net AUD_DIV_L: now also C61.1, R36.2, R37.1; no longer C63.1, R37.2, R38.1
- net AUD_DIV_R: now also C63.1, R38.2, R39.1; no longer C65.1, R39.2, R40.1
- net AUD_VINL: now also C62.2; no longer C63.2
- net AUD_VINR: now also C64.2; no longer C65.2
- net AV_AVDD: now also C18.1, C53.1; no longer C19.1, C55.1
- net AV_C0: now also R20.1; no longer R21.1
- net AV_C1: now also R19.1; no longer R20.1
- net AV_C5: now also R18.1; no longer R19.1
- net AV_C6: now also R17.1; no longer R18.1
- net AV_C7: now also R16.1; no longer R17.1
- net AV_DE: now also R23.1; no longer R24.1
- net AV_DVDD: now also C16.1, C47.1; no longer C17.1, C51.1
- net AV_DVDDIO: now also C19.1, C43.1, R27.1; no longer C20.1, C47.1, R30.1
- net AV_HS: now also R21.1; no longer R22.1
- net AV_PVDD: now also C17.1, C41.2, C51.1; no longer C18.1, C43.2, C53.1
- net AV_VS: now also R22.1; no longer R23.1
- net CAPC2: now also C34.1; no longer C37.1
- net CAPY1: now also C31.1; no longer C34.1
- net CAPY2: now also C29.1, C31.2; no longer C31.1, C37.2
- net CML: now also C39.1; no longer C41.1
- net ELPF: now also C42.1, R15.1; no longer C43.1, R16.1
- net ELPF_RC: now also C41.1, R15.2; no longer C42.1, R16.2
- net FB_1V8A: now also C12.2, R7.2, R8.1; no longer C13.2, R8.2, R9.1
- net FB_1V8B: now also C15.2, R10.1, R9.2; no longer C16.2, R10.2, R11.1
- net FB_3V3: now also C9.2, R5.2, R6.1; no longer C6.2, R3.2, R4.1
- net FMT: now also R35.1; no longer R36.1
- net GND: now also C13.2, C16.2, C27.2, C37.2, C43.2, C63.2, C65.2, R10.2, R26.2, R30.2, R37.2, R39.2, R44.2, R48.2, R51.2, R8.2, U11.3 (GND), U11.8 (GND); no longer C12.2, C15.2, C23.2, C31.2, C41.2, C62.2, C64.2, R14.2, R27.2, R36.2, R38.2, R40.2, R45.2, R49.2, R9.2
- net HDMI_5V: now also C76.1, R49.1; no longer R51.1
- net HDMI_HPD: now also R51.1
- net HDMI_SCL: now also R49.2; no longer R50.2
- net HDMI_SDA: now also R50.2; no longer R51.2
- net IN_C0: now also R20.2; no longer R21.2
- net IN_C1: now also R19.2; no longer R20.2
- net IN_C5: now also R18.2; no longer R19.2
- net IN_C6: now also R17.2; no longer R18.2
- net IN_C7: now also R16.2; no longer R17.2
- net IN_DE: now also R23.2; no longer R24.2
- net IN_HS: now also R21.2; no longer R22.2
- net IN_INT: now also R27.2; no longer R28.2
- net IN_RESET_N: now also R26.1; no longer R27.1
- net IN_SCL: now also R24.2; no longer R25.2
- net IN_SDA: now also R25.2; no longer R26.2
- net IN_VS: now also R22.2; no longer R23.2
- net MD0: now also R33.1; no longer R34.1
- net MD1: now also R34.1; no longer R35.1
- net OUT_I2S0: now also R43.1; no longer R44.1
- net OUT_INT: now also R47.2; no longer R48.2
- net OUT_LRCLK: now also R42.1; no longer R43.1
- net OUT_MCLK: now also R40.1; no longer R41.1
- net OUT_PD: now also R48.1; no longer R49.1
- net OUT_SCL: now also R45.2; no longer R46.2
- net OUT_SCLK: now also R41.1; no longer R42.1
- net OUT_SDA: now also R46.2; no longer R47.2
- net PD_FB: now also R30.1; no longer R31.1
- net PD_HS_IN_CS_IN: now also R31.1; no longer R32.1
- net PD_VS_IN: now also R32.1; no longer R33.1
- net PWRDWN: now also R29.2; no longer R30.2
- net RCA_L: now also R36.1; no longer R37.1
- net RCA_PB: now also C24.1, R12.1, U11.2 (D1-), U11.9 (NC); no longer C25.1, R13.1
- net RCA_PR: now also C25.1, R13.1, U11.4 (D2+), U11.7 (NC); no longer C26.1, R14.1
- net RCA_R: now also R38.1; no longer R39.1
- net RCA_Y: now also C23.1, C26.1, R11.1, U11.1 (D1+), U11.10 (NC); no longer C24.1, C27.1, R12.1
- net REFOUT: now also C37.1; no longer C39.1
- net R_EXT: now also R44.1; no longer R45.1
- net SYNC_Y: now also C26.2; no longer C27.2
- net TX_AVDD: now also C21.1, C69.1; no longer C22.1, C73.1
- net TX_DVDD: now also C20.1, C65.1; no longer C21.1, C69.1
- net TX_I2S0: now also R43.2; no longer R44.2
- net TX_LRCLK: now also R42.2; no longer R43.2
- net TX_MCLK: now also R40.2; no longer R41.2
- net TX_PLVDD: now also C22.1, C73.1; no longer C23.1, C75.1
- net TX_SCLK: now also R41.2; no longer R42.2
- net VREF: now also C55.1; no longer C57.1
- net XTAL: now also C27.1, R14.1; no longer C28.1, R15.1
- net XTAL1: now also C28.1, R14.2; no longer C29.1, R15.2
- removed net 2V5: C11.1, C14.1, C8.1, C9.1, L1.2, R5.1, R7.1, U6.3 (IN), U7.3 (IN)
- removed net EN_1V8: C10.1, R7.2, U6.2 (EN), U7.2 (EN)
- removed net FB_2V5: C9.2, R5.2, R6.1, U4.5 (FB)
- net SW_2V5 renamed SW_3V6
- new net 3V6: C5.1, C6.1, C7.1, L1.2, R3.1, U5.2 (EN), U5.3 (IN)
- new net FB_3V6: C6.2, R3.2, R4.1, U4.5 (FB)
- no-connect marks 20 -> 22
Other:
- moved on the sheet: C10, C11, C12, C13, C14, C15, C16, C17, C18, C19, C20, C21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
