File: hardware/av-board/rev-ca/av-board-ca.kicad_sch (KiCad schematic)
At the start: 280 parts, among them J1 RCA Y, J11 XIAO 5V..D7, J12 XIAO D0..D6, J13 OPTICAL, J14 RCA S/PDIF, J15 USB-C 5V, J16 JTAG, J2 RCA Pb, J20 DF40HC(3.0)-80DS, J21 DF40HC(3.0)-100DS, J22 DF40HC(3.0)-100DS, J3 RCA Pr, J4 RCA L, J5 RCA R, J6 HDMI-001, J7 SYNC, J8 VGA, Q1 2N7002, Q2 2N7002, Q3 2N7002, Q4 2N7002, SW1 TS-1187A-B-A-B, SW2 TS-1187A-B-A-B, SW3 TS-1187A-B-A-B, U1 ADV7181DBCPZ-RL, U10 TPD4E05U06DQAR, U12 TPS7A2045PDBVR, U13 SN74LVC1GU04DBVR, U14 SN74LVC1G04DBVR, U15 SN74LVC1G04DBVR, U17 MS5351M, U19 TPD4E05U06DQAR, U2 ADV7511KSTZ, U20 TPD4E05U06DQAR, U21 SN74LVC2G17DBVR, U22 SN74LVC8T245PWR, U23 SN74AVC4T245PWR, U24 ME6211C30M5G-N, U3 PCM1808PWR, U4 TLV62569DBVR, U5 TPS7A7001DDAR, U6 TPS7A7001DDAR, U7 TPS7A7001DDAR, U8 TPD4E05U06DQAR, U9 TPD4E05U06DQAR, Y1 28.63636MHz 20pF, Y2 25MHz 10pF

Commit message: AV boards: the last complete, valid design of each revision; decoupling at the pins
Each revision's board, schematic, fab files and renders are its last complete
route: DRC clean, no unconnected items, ERC clean, the board equal to its
schematic part for part (pads, values, footprints; only the mounting holes
H1-H4 have no symbol).

- Rev A: the silkscreen pass (labels clear of pads, texts and part bodies);
  copper unchanged.
- Rev B: the previous route with the silkscreen pass. Its schematic stays the
  one it was routed from: board.py now numbers eight capacitors the other way
  round, and its placement fixes (below) are not routed yet, the routes on the
  new placement having left 1 and 3 connections (review.md, Status).
- C-A: routed again on the fixed placement (try-ca-p1), the copper the router
  laid twice over taken up (218 segments).
- C-B: S/PDIF on rev B's 5-pin header instead of the coax jack, the HDMI
  receptacle next to the RCAs, the board 100 x 100 mm; routed again on the
  fixed placement (try-cb-p3). 5.4 mm of copper laid side by side in five
  nets is left (rev-c/review.md).

The review found decoupling not at the pins on every board (ADV7511 9-25 mm,
DP159 6-13 mm, the bucks' input capacitor by EN, the LDOs' capacitors, the
clock LDOs 73-80 mm from their chip) and C's VBUS_IN 0.25 mm wide for 2 A:
- parts.py: Part.at = "REF.PAD", the one pad a capacitor or filter serves;
  circuits, carrier.py and board.py name it for every regulator and supply pin
- pcbkit.py placer: ESD parts first, then small chips, then the at= capacitors
  and bias parts in board.py order; mean pin-to-capacitor distance on the
  placements: rev B 8.1 -> 3.6 mm, C-A 6.3 -> 3.3, C-B 5.5 -> 3.4
- rev C: VBUS_IN 0.7/1.2 mm into the TVS and fuse; rev B and C: the coax
  slicer placed first (SPDIF_AC a bias net); rev B: the buck U4 turned over

Kit: the silkscreen pass (labels clear of pads, texts, parts and the SOM,
reserved in the placer); prune takes up copper lying on another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
Parts:
- C11, C14, C8: value 10u -> 220p; footprint Capacitor_SMD:C_0805_2012Metric -> Capacitor_SMD:C_0402_1005Metric; LCSC C15850 -> C1530
- C12, C15, C9: value 220p -> 10u; footprint Capacitor_SMD:C_0402_1005Metric -> Capacitor_SMD:C_0805_2012Metric; LCSC C1530 -> C15850
- C5: value 10u -> 6.8p; footprint Capacitor_SMD:C_0805_2012Metric -> Capacitor_SMD:C_0402_1005Metric; LCSC C15850 -> C1576
- C6: value 6.8p -> 10u; footprint Capacitor_SMD:C_0402_1005Metric -> Capacitor_SMD:C_0805_2012Metric; LCSC C1576 -> C15850
Connections:
- net FB_1V8A: now also C11.2; no longer C12.2
- net FB_1V8B: now also C14.2; no longer C15.2
- net FB_3V3: now also C8.2; no longer C9.2
- net FB_3V6: now also C5.2; no longer C6.2
- net GND: now also C12.2, C15.2, C6.2, C9.2; no longer C11.2, C14.2, C5.2, C8.2
Other:
- moved on the sheet: C10, C11, C12, C13, C14, C15, C5, C6, C7, C8, C81, C82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

Commit message: AV board C-B: a protected debug header and test pads; the kit on KiCad 10, a second host
C-B (the SOM hides the FPGA's pins, so the board brings out what bring-up needs):
- J17, a 2 x 8 header left of the SOM: the ADV7181D's, the DP159's and the MS5351M's I2C, six
  spare FPGA pins, J22's nearest (dbg0-dbg5: AB16 L13 M13 AA16 AB17 Y17, LVCMOS33 in
  fpga/av-board-cb.cst), a 3.3 V reference and ground, labelled pin by pin, "DEBUG" above it.
  Every pin but ground through 220 R by the header (C25091, as Digilent's Pmod ports): a slipped
  probe or a wrong wire drives at most 15 mA into a pin; VREF, beside ground, is a reference
  (50 mW in its resistor when shorted), not a supply.
- A bare test pad on each rail by its regulator (+5V 3V6 3V3 1V8 1V1 3V0 2V5 5VA), labelled,
  and two ground pads with holes for a wire loop. Not assembled.
- The DP159's ground pins 19 and 41 now reach into its exposed pad: their fanout stubs stopped
  0.22 mm short of it, the prune pass took them up, and pin 19 was left open
  (gen_pcb.py serdes()).
- Re-routed: the best of a batch (v5): DRC 0 errors, 0 unconnected; schematic = board.py =
  board (1064 pins); fab files, renders and rev-c/review.md's layout numbers updated. Three
  resistors after the debug block are renumbered (R100-R102 -> R113-R115).
- Known, fixes next: an HDMI 2.0 layout audit against TI's SN65DP159 and SPRAAR7 guidelines
  finds other nets' vias against the TMDS run (their plane antipads within 0.01-0.21 mm),
  pairs 3W apart (TI: 5W), the transceivers' reference clock autorouted as two single lines,
  a crystal and a mounting hole near the lines, and no plane voids under the pads on them.

rev-c/review.md: kit/xtalk.py measures analog tracks against digital tracks only; KiCad's DRC
with the 0.5 mm rule as a custom rule counts vias too, and finds two of RCA_SYNC's vias 0.27 mm
from the VGA DDC clock on C-A (the C-A text said nothing but XTAL1/LLC came that close).

Kit:
- main(): the board made with its project (pcbn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
Parts:
- SO1, SO2, SO3, SO4: now left out of the parts list
Changed lines of the file:
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@@
     (unit 1)
     (exclude_from_sim no)
-    (in_bom yes)
+    (in_bom no)
     (on_board yes)
     (dnp no)
@@
     (unit 1)
     (exclude_from_sim no)
-    (in_bom yes)
+    (in_bom no)
     (on_board yes)
     (dnp no)
@@
     (unit 1)
     (exclude_from_sim no)
-    (in_bom yes)
+    (in_bom no)
     (on_board yes)
     (dnp no)
@@
     (unit 1)
     (exclude_from_sim no)
-    (in_bom yes)
+    (in_bom no)
     (on_board yes)
     (dnp no)
